File: control_boad_2021-2/control_boad_2021-2.sch (KiCad schematic (older format))
At the start: 6 parts, among them J1 Conn_01x10_Female, J2 Conn_01x10_Female, J3 Conn_01x02, U1 ESP32-DevKitC, U2 IM920s

Commit message: complete!!!
Parts:
- added D1, D2: LED, LED_SMD:LED_0603_1608Metric, symbol Device:LED
- added D3, D4, D5: WS2812B, LED_SMD:LED_WS2812B_PLCC4_5.0x5.0mm_P3.2mm, symbol LED:WS2812B
- added H1, H2, H3, H4: MountingHole, MountingHole:MountingHole_3.2mm_M3_Pad_Via, symbol Mechanical:MountingHole
- added H10, H9: MountingHole, MountingHole:MountingHole_3.2mm_M3_Pad, symbol Mechanical:MountingHole
- added H5, H6, H7, H8: MountingHole_Pad, MountingHole:MountingHole_3.2mm_M3_Pad, symbol Mechanical:MountingHole_Pad
- added J4: Conn_01x02, Connector_USB_additional:USB micro B 2pin, symbol Connector_Generic:Conn_01x02
- added J5: Conn_01x03_Female, Connector_JST:JST_XA_B03B-XASK-1_1x03_P2.50mm_Vertical, symbol Connector:Conn_01x03_Female
- added R1, R2: R, Resistor_SMD:R_0603_1608Metric, symbol Device:R
Connections:
- net +5V: now also J4.1 (Pin_1)
- net GND: now also H5.1, H6.1, H7.1, H8.1, J4.2 (Pin_2), R1.2, R2.2
- net im920_status: now also D1.2 (A)
- net im920s_xmit: now also D2.2 (A)
- new net: D3.2 (DOUT), D4.4 (DIN)
- new net: D4.2 (DOUT), D5.4 (DIN)
- new net: D1.1 (K), R1.1
- new net: D2.1 (K), R2.1
- new net +5VA: D3.1 (VDD), D4.1 (VDD), D5.1 (VDD), J5.1 (Pin_1)
- new net GNDA: D3.3 (VSS), D4.3 (VSS), D5.3 (VSS), J5.3 (Pin_3)
- new net datain: D3.4 (DIN), J5.2 (Pin_2)
