File: control_boad_2021-2/control_boad_2021-2.kicad_pcb (KiCad board)
At the start: 2 copper layers, 6 parts, among them J1 Conn_01x10_Female, J2 Conn_01x10_Female, J3 Conn_01x02, U1 ESP32-DevKitC, U2 IM920s

Commit message: complete!!!
Parts:
- added D1: LED, LED_SMD:LED_0603_1608Metric, F.Cu at (118.7, 57.8)
- added D2: LED, LED_SMD:LED_0603_1608Metric, F.Cu at (127.6, 57.8)
- added D3: WS2812B, LED_SMD:LED_WS2812B_PLCC4_5.0x5.0mm_P3.2mm, B.Cu at (155.6, 76.2)
- added D4: WS2812B, LED_SMD:LED_WS2812B_PLCC4_5.0x5.0mm_P3.2mm, B.Cu at (155.6, 91.4)
- added D5: WS2812B, LED_SMD:LED_WS2812B_PLCC4_5.0x5.0mm_P3.2mm, B.Cu at (155.6, 106.7)
- added H1: MountingHole, MountingHole:MountingHole_3.2mm_M3_Pad_Via, F.Cu at (69.2, 57.8)
- added H10: MountingHole, MountingHole:MountingHole_3.2mm_M3_Pad, F.Cu at (155.6, 118.1)
- added H2: MountingHole, MountingHole:MountingHole_3.2mm_M3_Pad_Via, F.Cu at (69.2, 142.9)
- added H3: MountingHole, MountingHole:MountingHole_3.2mm_M3_Pad_Via, F.Cu at (137.8, 142.9)
- added H4: MountingHole, MountingHole:MountingHole_3.2mm_M3_Pad_Via, F.Cu at (137.8, 57.8)
- added H5: MountingHole_Pad, MountingHole:MountingHole_3.2mm_M3_Pad, F.Cu at (69.2, 76.2)
- added H6: MountingHole_Pad, MountingHole:MountingHole_3.2mm_M3_Pad, F.Cu at (69.2, 124.5)
- added H7: MountingHole_Pad, MountingHole:MountingHole_3.2mm_M3_Pad, F.Cu at (95.9, 63.5)
- added H8: MountingHole_Pad, MountingHole:MountingHole_3.2mm_M3_Pad, F.Cu at (95.9, 137.2)
- added H9: MountingHole, MountingHole:MountingHole_3.2mm_M3_Pad, F.Cu at (155.6, 57.8)
- added J4: Conn_01x02, Connector_USB_additional:USB micro B 2pin, F.Cu at (108.0, 57.1)
- added J5: Conn_01x03_Female, Connector_JST:JST_XA_B03B-XASK-1_1x03_P2.50mm_Vertical, F.Cu at (153.1, 67.3)
- added R1: R, Resistor_SMD:R_0603_1608Metric, F.Cu at (108.0, 70.5)
- added R2: R, Resistor_SMD:R_0603_1608Metric, F.Cu at (111.1, 70.5)
- moved JP1 64.3 mm to (106.7, 78.7)
- moved J3 48.4 mm to (108.0, 143.5), turned to 180 degrees
- moved J2 45.0 mm to (95.2, 88.9)
- moved J1 45.0 mm to (69.8, 88.9)
- moved U2 28.3 mm to (130.8, 71.8), turned to 270 degrees
- moved U1 10.6 mm to (130.2, 108.6), turned to 180 degrees
Routing:
- net +5V: track 0.00 -> 146.9 mm, vias 0 -> 3
- net +3V3: track 0.00 -> 125.5 mm, vias 0 -> 2
- net digital8_io33: track 0.00 -> 107.7 mm, vias 0 -> 2
- net analog0_io25: track 0.00 -> 103.1 mm, vias 0 -> 2
- net digital7_io32: track 0.00 -> 93.5 mm, vias 0 -> 1
- net digital1_io14: track 0.00 -> 90.6 mm, vias 0 -> 2
- net analog2_io39: track 0.00 -> 88.6 mm, vias 0 -> 2
- net anarog1_io36: track 0.00 -> 88.3 mm, vias 0 -> 2
- net digital0_io13: track 0.00 -> 87.0 mm, vias 0 -> 2
- net serial1_RX_io26: track 0.00 -> 80.2 mm, vias 0 -> 1
- net serial1_TX_io27: track 0.00 -> 79.2 mm, vias 0 -> 1
- net digital2_io18: track 0.00 -> 58.4 mm
- net digital6_io23: track 0.00 -> 57.9 mm
- net digital5_io22: track 0.00 -> 57.9 mm
- net digital3_io19: track 0.00 -> 57.4 mm
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- added copper zone on B.Cu, net GND
- added copper zone on F.Cu, net GND
- added copper zone on B.Cu, net GNDA
- added copper zone on F.Cu, net GNDA
Other:
- board outline added: 95.9 x 92.7 mm
- board text added: "status"
- board text added: "xmit"

Commit message: added gbr files
Other:
- board text added: "CB-2021-2"
- board text added: "designed by paripal"
Changed lines of the file:
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@@
-(kicad_pcb (version 20171130) (host pcbnew "(5.1.4)-1")
+(kicad_pcb (version 20171130) (host pcbnew "(5.1.5)-3")
   (general
     (thickness 1.6)
-    (drawings 26)
+    (drawings 25)
     (tracks 380)
     (zones 0)
@@
   )
   (setup
-    (last_trace_width 0.75)
+    (last_trace_width 0.25)
     (user_trace_width 0.5)
     (user_trace_width 0.75)
@@
       (outputformat 1)
       (mirror false)
-      (drillshape 1)
+      (drillshape 0)
       (scaleselection 1)
-      (outputdirectory ""))
+      (outputdirectory "control_boad_2021-2/"))
   )
   (net 0 "")
@@
     )
   )
+  (gr_text "designed by paripal" (at 83.82 133.35 90) (layer F.SilkS)
+    (effects (font (size 1 1) (thickness 0.15)))
+  )
+  (gr_text "CB-2021-2\n" (at 81.28 133.35 90) (layer F.SilkS)
+    (effects (font (size 1.5 1.5) (thickness 0.2)))
+  )
   (gr_line (start 147.32 107.315) (end 147.32 142.875) (layer Edge.Cuts) (width 0.05))
   (gr_line (start 149.86 118.11) (end 149.86 107.315) (layer Edge.Cuts) (width 0.05))
@@
   (gr_line (start 161.29 57.785) (end 161.29 118.11) (layer Edge.Cuts) (width 0.05))
   (gr_line (start 149.86 57.785) (end 149.86 69.85) (layer Edge.Cuts) (width 0.05))
-  (dimension 81.915 (width 0.12) (layer F.SilkS)
-    (gr_text "81.915 mm" (at 106.3625 157.48) (layer F.SilkS)
-      (effects (font (size 1 1) (thickness 0.15)))
-    )
-    (feature1 (pts (xy 147.32 146.685) (xy 147.32 156.796421)))
-    (feature2 (pts (xy 65.405 146.685) (xy 65.405 156.796421)))
-    (crossbar (pts (xy 65.405 156.21) (xy 147.32 156.21)))
-    (arrow1a (pts (xy 147.32 156.21) (xy 146.193496 156.796421)))
-    (arrow1b (pts (xy 147.32 156.21) (xy 146.193496 155.623579)))
-    (arrow2a (pts (xy 65.405 156.21) (xy 66.531504 156.796421)))
-    (arrow2b (pts (xy 65.405 156.21) (xy 66.531504 155.623579)))
-  )
   (gr_line (start 147.32 57.785) (end 147.32 69.85) (layer Edge.Cuts) (width 0.05))
   (gr_arc (start 143.51 57.785) (end 147.32 57.785) (angle -90) (layer Edge.Cuts) (width 0.05))
@@
   )
   (gr_line (start 114.935 145.415) (end 114.935 55.88) (layer F.SilkS) (width 0.12))
-  (dimension 76.2 (width 0.12) (layer F.SilkS)
-    (gr_text "76.200 mm" (at 103.505 152.4) (layer F.SilkS)
-      (effects (font (size 1 1) (thickness 0.15)))
-    )
-    (feature1 (pts (xy 141.605 146.685) (xy 141.605 151.716421)))
-    (feature2 (pts (xy 65.405 146.685) (xy 65.405 151.716421)))
-    (crossbar (pts (xy 65.405 151.13) (xy 141.605 151.13)))
-    (arrow1a (pts (xy 141.605 151.13) (xy 140.478496 151.716421)))
-    (arrow1b (pts (xy 141.605 151.13) (xy 140.478496 150.543579)))
-    (arrow2a (pts (xy 65.405 151.13) (xy 66.531504 151.716421)))
-    (arrow2b (pts (xy 65.405 151.13) (xy 66.531504 150.543579)))
-  )
-  (dimension 92.71 (width 0.12) (layer F.SilkS)
-    (gr_text "92.710 mm" (at 59.055 100.33 270) (layer F.SilkS)
-      (effects (font (size 1 1) (thickness 0.15)))
-    )
-    (feature1 (pts (xy 65.405 146.685) (xy 59.738579 146.685)))
-    (feature2 (pts (xy 65.405 53.975) (xy 59.738579 53.975)))
-    (crossbar (pts (xy 60.325 53.975) (xy 60.325 146.685)))
-    (arrow1a (pts (xy 60.325 146.685) (xy 59.738579 145.558496)))
-    (arrow1b (pts (xy 60.325 146.685) (xy 60.911421 145.558496)))
-    (arrow2a (pts (xy 60.325 53.975) (xy 59.738579 55.101504)))
-    (arrow2b (pts (xy 60.325 53.975) (xy 60.911421 55.101504)))
-  )
   (gr_arc (start 69.215 142.875) (end 65.405 142.875) (angle -90) (layer Edge.Cuts) (width 0.05))
   (gr_arc (start 69.215 57.785) (end 69.215 53.975) (angle -90) (layer Edge.Cuts) (width 0.05))

Commit message: v2 comp
Parts:
- added R3: R, Resistor_SMD:R_0603_1608Metric, F.Cu at (106.0, 134.6)
- added R4: R, Resistor_SMD:R_0603_1608Metric, F.Cu at (108.0, 134.6)
- added R5: R, Resistor_SMD:R_0603_1608Metric, F.Cu at (108.0, 66.0)
- added R6: R, Resistor_SMD:R_0603_1608Metric, F.Cu at (106.0, 66.0)
- J3, J4: value Conn_01x02 -> USB_C_Receptacle_PowerOnly_6P; footprint Connector_USB_additional:USB micro B 2pin -> Connector_USB_additional:USB_C_Receptacle_CUI_ UJC-HP-3-SMT-TR_TopMnt_Horizontal
- moved J3 3.24 mm to (107.3, 146.7), turned to 0 degrees
- moved J4 3.24 mm to (107.3, 54.0), turned to 180 degrees
Connections:
- D3 pad 1: +5VA -> +5V
- D3 pad 3: GNDA -> GND
- D4 pad 1: +5VA -> +5V
- D4 pad 3: GNDA -> GND
- D5 pad 1: +5VA -> +5V
- D5 pad 2: Net-(D5-Pad2) -> unconnected-(D5-DOUT-Pad2)
- D5 pad 3: GNDA -> GND
- J2 pad 8: serial1_RX_io26 -> datain
- J5 pad 1: +5VA -> +5V
- J5 pad 3: GNDA -> GND
- U1 pad 10: serial1_RX_io26 -> datain
- U1 pad 13: Net-(U1-Pad13) -> unconnected-(U1-IO12-Pad13)
- U1 pad 16: Net-(U1-Pad16) -> unconnected-(U1-SD2-Pad16)
- U1 pad 17: Net-(U1-Pad17) -> unconnected-(U1-SD3-Pad17)
- U1 pad 18: Net-(U1-Pad18) -> unconnected-(U1-CMD-Pad18)
- U1 pad 2: Net-(U1-Pad2) -> unconnected-(U1-EN-Pad2)
- U1 pad 29: Net-(U1-Pad29) -> unconnected-(U1-IO5-Pad29)
- U1 pad 32: Net-(U1-Pad32) -> unconnected-(U1-IO4-Pad32)
- U1 pad 33: Net-(U1-Pad33) -> unconnected-(U1-IO0-Pad33)
- U1 pad 34: Net-(U1-Pad34) -> unconnected-(U1-IO2-Pad34)
- U1 pad 35: Net-(U1-Pad35) -> unconnected-(U1-IO15-Pad35)
- U1 pad 36: Net-(U1-Pad36) -> unconnected-(U1-SD1-Pad36)
- U1 pad 37: Net-(U1-Pad37) -> unconnected-(U1-SD0-Pad37)
- U1 pad 38: Net-(U1-Pad38) -> unconnected-(U1-CLK-Pad38)
- U1 pad 5: Net-(U1-Pad5) -> unconnected-(U1-IO34-Pad5)
- U1 pad 6: Net-(U1-Pad6) -> unconnected-(U1-IO35-Pad6)
- U2 pad 10: Net-(U2-Pad10) -> unconnected-(U2-IO10-Pad10)
- U2 pad 11: Net-(U2-Pad11) -> unconnected-(U2-NC-Pad11)
- U2 pad 12: Net-(U2-Pad12) -> unconnected-(U2-NC-Pad12)
- U2 pad 13: Net-(U2-Pad13) -> unconnected-(U2-NC-Pad13)
- U2 pad 14: Net-(U2-Pad14) -> unconnected-(U2-NC-Pad14)
- U2 pad 16: Net-(U2-Pad16) -> unconnected-(U2-REG-Pad16)
- U2 pad 19: Net-(U2-Pad19) -> unconnected-(U2-RESET-Pad19)
- U2 pad 2: Net-(U2-Pad2) -> unconnected-(U2-IO2-Pad2)
- U2 pad 20: Net-(U2-Pad20) -> unconnected-(U2-RSV-Pad20)
- U2 pad 4: Net-(U2-Pad4) -> unconnected-(U2-IO4/SLEEP-Pad4)
- U2 pad 5: Net-(U2-Pad5) -> unconnected-(U2-IO5-Pad5)
- U2 pad 8: Net-(U2-Pad8) -> unconnected-(U2-IO8-Pad8)
- U2 pad 9: Net-(U2-Pad9) -> unconnected-(U2-IO9-Pad9)
Routing:
- net datain: track 7.10 -> 132.0 mm, vias 0 -> 3
- net serial1_RX_io26: track 80.2 -> 0.00 mm, vias 1 -> 0
- net +5V: track 146.9 -> 226.9 mm, vias 3 -> 7
- net +5VA: track 45.3 -> 0.00 mm
- net Net-(J3-CC1): track 0.00 -> 5.15 mm
- net Net-(J4-CC2): track 0.00 -> 5.15 mm
- net Net-(J3-CC2): track 0.00 -> 4.89 mm
- net Net-(J4-CC1): track 0.00 -> 4.89 mm
- net GND: track 3.15 -> 7.23 mm, vias 102 -> 126
- net GNDA: vias 14 -> 0
- removed copper zone on B.Cu, net GNDA
- removed copper zone on F.Cu, net GNDA
Other:
- net class Default removed
- board text added: "CB-2021-2_v2"
- board text removed: "CB-2021-2"
