File: control_interface_boad_2021-2/control_interface_boad_2021-2.sch (KiCad schematic (older format))
At the start: 6 parts

Commit message: complete!!!
Parts:
- added D1, D2, D3, D4, D5: WS2812B, LED_SMD:LED_WS2812B_PLCC4_5.0x5.0mm_P3.2mm, symbol LED:WS2812B
- added H1, H2, H3, H4, H5, H6, H7, H8: MountingHole_Pad, MountingHole:MountingHole_3.2mm_M3_Pad, symbol Mechanical:MountingHole_Pad
- added J10, J11, J12, J15, J16, J17, J18, J6, J9: Conn_01x03_Female, Connector_JST:JST_XA_S03B-XASK-1_1x03_P2.50mm_Horizontal, symbol Connector:Conn_01x03_Female
- added J13, J14: Conn_01x04_Female, Connector_JST:JST_XA_S04B-XASK-1_1x04_P2.50mm_Horizontal, symbol Connector:Conn_01x04_Female
- added J3: Conn_01x02_Female, Connector_JST:JST_XA_S02B-XASK-1_1x02_P2.50mm_Horizontal, symbol Connector:Conn_01x02_Female
- added J4, J5: Conn_01x05_Female, Connector_JST:JST_XA_S05B-XASK-1_1x05_P2.50mm_Horizontal, symbol Connector:Conn_01x05_Female
- added J7, J8: Conn_01x10_Male, Connector_PinHeader_2.54mm:PinHeader_1x10_P2.54mm_Vertical, symbol Connector:Conn_01x10_Male
- J1, J2: renamed from J?; footprint (none) -> Connector_PinHeader_2.54mm:PinHeader_1x10_P2.54mm_Vertical
- SW1, SW2, SW3, SW4: renamed from SW?; footprint (none) -> Button_Switch_Keyboard:SW_Cherry_MX_1.25u_PCB
Connections:
- net +3V3: now also J4.2 (Pin_2)
- net +5V: now also J5.2 (Pin_2), J6.1 (Pin_1)
- net GND: now also H1.1, H2.1, H3.1, H4.1, J3.2 (Pin_2), J4.1 (Pin_1), J5.5 (Pin_5), J6.3 (Pin_3)
- net analog0 renamed analog0_stick_x
- net analog0_stick_x: now also J4.3 (Pin_3)
- net analog1 renamed analog1_stick_y
- net analog1_stick_y: now also J4.4 (Pin_4)
- net analog2 renamed analog2_pedal
- net digital0 renamed digital0_key0
- net digital1 renamed digital1_key1
- net digital2 renamed digital2_key2
- net digital3 renamed digital3_key3
- net digital4 renamed digital4_stick_sw
- net digital4_stick_sw: now also J4.5 (Pin_5)
- net digital5 renamed digital5_lmtsw
- net digital5_lmtsw: now also J3.1 (Pin_1)
- net digital6 renamed digital6_encoder_a
- net digital6_encoder_a: now also J5.3 (Pin_3)
- net digital7 renamed digital7_encoder_b
- net digital7_encoder_b: now also J5.1 (Pin_1)
- net digital8 renamed digital8_nc1
- net serial0_RX renamed serial0_RX_nc1
- net serial0_TX renamed serial0_TX_nc1
- net serial1_RX renamed serial1_RX_as_digital_neopixel
- net serial1_RX_as_digital_neopixel: now also J6.2 (Pin_2)
- net serial1_TX renamed serial1_TX_nc1
- new net: D1.2 (DOUT), D2.4 (DIN)
- new net: D2.2 (DOUT), D3.4 (DIN)
- new net: D3.2 (DOUT), D4.4 (DIN)
- new net: D4.2 (DOUT), D5.4 (DIN)
- new net +3.3VA: J8.2 (Pin_2)
- new net +5VA: D1.1 (VDD), D2.1 (VDD), D3.1 (VDD), D4.1 (VDD), D5.1 (VDD), J10.2 (Pin_2), J11.2 (Pin_2), J12.2 (Pin_2), J13.1 (Pin_1), J14.1 (Pin_1), J15.1 (Pin_1), J16.1 (Pin_1), J17.1 (Pin_1), J18.1 (Pin_1), J8.1 (Pin_1), J9.2 (Pin_2)
- new net GNDA: D1.3 (VSS), D2.3 (VSS), D3.3 (VSS), D4.3 (VSS), D5.3 (VSS), H5.1, H6.1, H7.1, H8.1, J10.3 (Pin_3), J11.3 (Pin_3), J12.3 (Pin_3), J13.4 (Pin_4), J14.4 (Pin_4), J15.3 (Pin_3), J16.3 (Pin_3), J17.3 (Pin_3), J18.3 (Pin_3), J7.10 (Pin_10), J8.10 (Pin_10), J9.3 (Pin_3)
- new net analog0_neopixel4: D1.4 (DIN), J8.3 (Pin_3)
- new net analog1_nc2: J8.4 (Pin_4)
- new net analog2_nc2: J8.5 (Pin_5)
- new net digital0_sv0: J7.1 (Pin_1), J9.1 (Pin_1)
- new net digital1_sv1: J10.1 (Pin_1), J7.2 (Pin_2)
- new net digital2_sv2: J11.1 (Pin_1), J7.3 (Pin_3)
- new net digital3_sv3: J12.1 (Pin_1), J7.4 (Pin_4)
- new net digital4_neopixel0: J15.2 (Pin_2), J7.5 (Pin_5)
- new net digital5_neopixel1: J16.2 (Pin_2), J7.6 (Pin_6)
- new net digital6_neopixel2: J17.2 (Pin_2), J7.7 (Pin_7)
- new net digital7_neopixel3: J18.2 (Pin_2), J7.8 (Pin_8)
- new net digital8_nc2: J7.9 (Pin_9)
- new net serial0_RX_serial: J14.3 (Pin_3), J8.6 (Pin_6)
- new net serial0_TX_serial: J14.2 (Pin_2), J8.7 (Pin_7)
- new net serial1_RX_CAN: J13.3 (Pin_3), J8.8 (Pin_8)
- new net serial1_TX_CAN: J13.2 (Pin_2), J8.9 (Pin_9)
Other:
- note added: "encoder"
- note added: "lmtsw"
- note added: "stick"
- moved on the sheet: J1, J2, SW1, SW2, SW3, SW4
