File: control_interface_boad_2021-2/control_interface_boad_2021-2.kicad_pcb (KiCad board)
At the start: 2 copper layers, 97.2 x 99.1 mm, 35 parts, among them J1 Conn_01x10_Male, J10 Conn_01x03_Female, J11 Conn_01x03_Female, J12 Conn_01x03_Female, J13 Conn_01x04_Female, J14 Conn_01x04_Female, J15 Conn_01x03_Female, J16 Conn_01x03_Female, J17 Conn_01x03_Female, J18 Conn_01x03_Female, J2 Conn_01x10_Male, J3 Conn_01x02_Female, J4 Conn_01x05_Female, J5 Conn_01x05_Female, J6 Conn_01x03_Female, J7 Conn_01x10_Male, J8 Conn_01x10_Male, J9 Conn_01x03_Female, SW1 SW_Push, SW2 SW_Push, SW3 SW_Push, SW4 SW_Push

Commit message: v2 comp
Parts:
- added C1: 0.1u, Capacitor_SMD:C_0603_1608Metric, F.Cu at (139.7, 102.9)
- added J19: Conn_01x02_Pin, Connector_PinHeader_2.54mm:PinHeader_1x02_P2.54mm_Vertical, F.Cu at (118.1, 102.9)
- added R1: 10k, Resistor_SMD:R_0603_1608Metric, F.Cu at (129.5, 108.0)
- added R2: 120, Resistor_SMD:R_0603_1608Metric, F.Cu at (124.5, 106.7)
- added U1: MCP2551-I-SN, Package_SO:SOIC-8_3.9x4.9mm_P1.27mm, F.Cu at (133.3, 102.9)
- moved J13 0.16 mm to (117.0, 109.3)
Connections:
- D1 pad 1: +5VA -> +5V
- D1 pad 3: GNDA -> GND
- D2 pad 1: +5VA -> +5V
- D2 pad 3: GNDA -> GND
- D3 pad 1: +5VA -> +5V
- D3 pad 3: GNDA -> GND
- D4 pad 1: +5VA -> +5V
- D4 pad 3: GNDA -> GND
- D5 pad 1: +5VA -> +5V
- D5 pad 2: Net-(D5-Pad2) -> unconnected-(D5-DOUT-Pad2)
- D5 pad 3: GNDA -> GND
- H5 pad 1: GNDA -> GND
- H6 pad 1: GNDA -> GND
- H7 pad 1: GNDA -> GND
- H8 pad 1: GNDA -> GND
- J10 pad 2: +5VA -> +5V
- J10 pad 3: GNDA -> GND
- J11 pad 2: +5VA -> +5V
- J11 pad 3: GNDA -> GND
- J12 pad 2: +5VA -> +5V
- J12 pad 3: GNDA -> GND
- J13 pad 1: +5VA -> +5V
- J13 pad 2: serial1_TX_CAN -> /CANH
- J13 pad 3: serial1_RX_CAN -> /CANL
- J13 pad 4: GNDA -> GND
- J14 pad 1: +5VA -> +5V
- J14 pad 4: GNDA -> GND
- J15 pad 1: +5VA -> +5V
- J15 pad 3: GNDA -> GND
- J16 pad 1: +5VA -> +5V
- J16 pad 3: GNDA -> GND
- J17 pad 1: +5VA -> +5V
- J17 pad 3: GNDA -> GND
- J18 pad 1: +5VA -> +5V
- J18 pad 3: GNDA -> GND
- J5 pad 4: Net-(J5-Pad4) -> unconnected-(J5-Pin_4-Pad4)
- J7 pad 10: GNDA -> GND
- J8 pad 1: +5VA -> +5V
- J8 pad 10: GNDA -> GND
- J9 pad 2: +5VA -> +5V
- J9 pad 3: GNDA -> GND
Routing:
- net +5V: track 47.0 -> 330.5 mm, vias 0 -> 2
- net +5VA: track 241.8 -> 0.00 mm
- net /CANL: track 0.00 -> 29.5 mm
- net serial1_RX_CAN: track 43.5 -> 21.2 mm
- net /CANH: track 0.00 -> 17.3 mm
- net serial1_TX_CAN: track 36.9 -> 23.0 mm
- net Net-(J19-Pin_1): track 0.00 -> 7.10 mm
- net GND: track 0.00 -> 5.08 mm, vias 31 -> 95
- net Net-(U1-Rs): track 0.00 -> 4.48 mm
- net GNDA: vias 53 -> 0
- removed copper zone on B.Cu, net GNDA
- removed copper zone on F.Cu, net GNDA
Other:
- net class Default removed
- board text added: "CAN RX IO26 TX IO27"
- board text added: "CBIF-2021-2_v2 1/2"
- board text added: "CBIF-2021-2_v2 2/2"
- board text removed: "CBIF-2021-2 1/2"
- board text removed: "CBIF-2021-2 2/2"
- board text removed: "serial1 RX IO26 TX IO27"
